File: wifi_led_8266_driver.kicad_pcb (KiCad board)
At the start: 2 copper layers, 49.3 x 24.9 mm, 22 parts, among them J1 UART, J2 POWER, J3 WS2812B_DRIVER, SW1 RESET_BTN, SW2 BUTTON, SW3 FLASH_BTN, SW4 BOOT_BTN, U1 ESP-07, U2 MCP1825T

Commit message: propozycja
Parts:
- added J4: Conn_02x04_Odd_Even, Connector_PinHeader_1.27mm:PinHeader_2x04_P1.27mm_Vertical_SMD, B.Cu at (114.3, 92.7)
Connections:
- C1 pad 1: /5V_INP -> Net-(C1-Pad1)
- D1 pad 2: /5V_INP -> Net-(C1-Pad1)
- D2 pad 2: /5V_INP -> Net-(C1-Pad1)
- J2 pad 1: /5V_INP -> Net-(C1-Pad1)
- SW2 pad 2: GND -> Net-(SW2-Pad2)
- U1 pad 10: GND -> Net-(SW2-Pad2)
- U1 pad 4: Net-(U1-Pad4) -> /GPIO16
- U1 pad 5: Net-(U1-Pad5) -> /GPIO14
- U1 pad 6: Net-(U1-Pad6) -> /GPIO12
- U1 pad 7: Net-(U1-Pad7) -> /GPIO13
- U2 pad 1: /5V_INP -> Net-(C1-Pad1)
- U2 pad 2: /5V_INP -> Net-(C1-Pad1)
Routing:
- net Net-(SW2-Pad2): track 0.00 -> 7.95 mm
- net GND: track 135.5 -> 127.5 mm

Commit message: propozycja skonczona
Parts:
- moved J4 13.2 mm to (108.0, 81.2)
Connections:
- C1 pad 1: Net-(C1-Pad1) -> /5V_INP
- D1 pad 2: Net-(C1-Pad1) -> /5V_INP
- D2 pad 2: Net-(C1-Pad1) -> /5V_INP
- J2 pad 1: Net-(C1-Pad1) -> /5V_INP
- U2 pad 1: Net-(C1-Pad1) -> /5V_INP
- U2 pad 2: Net-(C1-Pad1) -> /5V_INP
Routing:
- net +3V3: track 47.6 -> 73.8 mm
- net /GPIO14: track 0.00 -> 15.8 mm, vias 0 -> 1
- net Net-(SW2-Pad2): track 7.95 -> 23.4 mm, vias 0 -> 1
- net /5V_INP: track 67.6 -> 80.7 mm, vias 1 -> 2
- net /GPIO12: track 0.00 -> 12.9 mm, vias 0 -> 1
- net /GPIO16: track 0.00 -> 9.86 mm, vias 0 -> 1
- net /GPIO13: track 0.00 -> 9.22 mm, vias 0 -> 1
- net GND: track 127.5 -> 119.6 mm, vias 9 -> 8

Commit message: wersja produkcyjna
Parts:
- J2: footprint Connector_PinHeader_2.54mm:PinHeader_1x02_P2.54mm_Vertical -> TerminalBlock_Phoenix:TerminalBlock_Phoenix_MPT-0,5-2-2.54_1x02_P2.54mm_Horizontal
- moved J2 2.52 mm to (102.9, 74.3), turned to 270 degrees
Routing:
- net GND: track 119.6 -> 131.6 mm, vias 8 -> 10
- net /5V_INP: track 80.7 -> 81.6 mm
Other:
- outline, holes or cut-outs redrawn
