File: wifi_led_8266_driver.sch (KiCad schematic (older format))
At the start: 1 part

Commit message: layout for enclouser https://www.tme.eu/pl/details/hm-1551usb3tsk/obudowy-uniwersalne/hammond/1551usb3tsk/
Parts:
- added C1: 4.7uF, Capacitor_SMD:C_1210_3225Metric, symbol Device:C_Small
- added C2: 1uF, Capacitor_SMD:C_0603_1608Metric_Pad1.05x0.95mm_HandSolder, symbol Device:C_Small
- added C3: 100nf, Capacitor_SMD:C_1206_3216Metric, symbol Device:C_Small
- added D1, D3: D, Diode_SMD:D_MiniMELF_Handsoldering, symbol Device:D
- added D2, D4: D, Diode_SMD:D_MELF_Handsoldering, symbol Device:D
- added D5: WS2812B, LED_SMD:LED_WS2812B_PLCC4_5.0x5.0mm_P3.2mm, symbol LED:WS2812B
- added J1: UART, Connector_PinHeader_2.54mm:PinHeader_1x03_P2.54mm_Vertical, symbol Connector:Conn_01x03_Male
- added J2: POWER, Connector_PinHeader_2.54mm:PinHeader_1x02_P2.54mm_Vertical, symbol Connector:Conn_01x02_Male
- added J3: WS2812B_DRIVER, Connector_PinHeader_2.54mm:PinHeader_1x03_P2.54mm_Vertical, symbol Connector:Conn_01x03_Male
- added R1, R2, R3: 10K, Resistor_SMD:R_1206_3216Metric, symbol Device:R_Small
- added R4: SB1, Resistor_SMD:R_0603_1608Metric, symbol Device:R_Small
- added R5: SB2, Resistor_SMD:R_0603_1608Metric, symbol Device:R_Small
- added SW1: RESET_BTN, Button_Switch_SMD:SW_SPST_B3S-1000, symbol Switch:SW_Push
- added SW2: BUTTON, Button_Switch_SMD:SW_SPST_B3S-1000, symbol Switch:SW_Push
- added SW3: FLASH_BTN, Button_Switch_SMD:SW_SPST_B3S-1000, symbol Switch:SW_Push
- added SW4: BOOT_BTN, Button_Switch_SMD:SW_SPST_B3S-1000, symbol Switch:SW_Push
- added U2: MCP1825T, Package_TO_SOT_SMD:SOT-223-6, symbol MCP1825T:MCP1825T
- gave numbers to parts that had none: 1
Connections:
- net labels added: +3.3V, 5V_INP, GND, GPIO0, GPIO2, RX, TX, WS2812B_DATA
- wire segments 0 -> 56
Other:
- note added: "Tutaj dwa złącza dla diod w razie czego wlutowac tylko jedną a drugie pady\n zewrzec chodzi o łączny spadek napięcia do 4.3V czyli 0.7V\n"

Commit message: propozycja
Parts:
- added J4: Conn_02x04_Odd_Even, Connector_PinHeader_1.27mm:PinHeader_2x04_P1.27mm_Vertical_SMD, symbol Connector_Generic:Conn_02x04_Odd_Even
Connections:
- net labels added: GPIO12, GPIO13, GPIO14, GPIO16
- wire segments 56 -> 69
Changed lines of the file:
@@
 Wire Wire Line
 	3150 1900 3150 1700
-Text Label 2450 1900 0    50   ~ 0
+Text Label 3000 4050 0    50   ~ 0
 5V_INP
 Wire Wire Line
@@
 L power:GND #PWR0111
 U 1 1 5B9E02BC
-P 2750 3850
-F 0 "#PWR0111" H 2750 3600 50  0001 C CNN
-F 1 "GND" H 2755 3677 50  0000 C CNN
-F 2 "" H 2750 3850 50  0001 C CNN
-F 3 "" H 2750 3850 50  0001 C CNN
-	1    2750 3850
+P 3000 4250
+F 0 "#PWR0111" H 3000 4000 50  0001 C CNN
+F 1 "GND" H 3005 4077 50  0000 C CNN
+F 2 "" H 3000 4250 50  0001 C CNN
+F 3 "" H 3000 4250 50  0001 C CNN
+	1    3000 4250
 	1    0    0    -1
 $EndComp
 Wire Wire Line
 	2400 3850 2750 3850
-Connection ~ 2750 3850
 Wire Wire Line
 	1200 3150 1200 2950
@@
 	3800 2950 3800 3350
 Connection ~ 3500 3350
+Wire Wire Line
+	2400 3550 2700 3550
+Wire Wire Line
+	2400 3650 2700 3650
+Wire Wire Line
+	2400 3750 2700 3750
+Wire Wire Line
+	2400 3950 2700 3950
+Text Label 2400 3550 0    50   ~ 0
+GPIO12
+Text Label 2400 3650 0    50   ~ 0
+GPIO13
+Text Label 2400 3750 0    50   ~ 0
+GPIO14
+Text Label 2400 3950 0    50   ~ 0
+GPIO16
+Text Label 3700 3950 0    50   ~ 0
+GPIO12
+Text Label 3700 4050 0    50   ~ 0
+GPIO13
+Text Label 3700 4150 0    50   ~ 0
+GPIO14
+Text Label 3700 4250 0    50   ~ 0
+GPIO16
+$Comp
+L Connector_Generic:Conn_02x04_Odd_Even J4
+U 1 1 5BA01931
+P 3400 4050
+F 0 "J4" H 3450 4367 50  0000 C CNN
+F 1 "Conn_02x04_Odd_Even" H 3450 4276 50  0000 C CNN
+F 2 "Connector_PinHeader_1.27mm:PinHeader_2x04_P1.27mm_Vertical_SMD" H 3400 4050 50  0001 C CNN
+F 3 "~" H 3400 4050 50  0001 C CNN
+	1    3400 4050
+	1    0    0    -1
+$EndComp
+Wire Wire Line
+	3200 4050 3000 4050
+Wire Wire Line
+	3000 3950 3200 3950
+Wire Wire Line
+	3200 4150 3000 4150
+Wire Wire Line
+	3200 4250 3000 4250
+Wire Wire Line
+	3700 4250 4000 4250
+Wire Wire Line
+	3700 4150 4000 4150
+Wire Wire Line
+	3700 4050 4000 4050
+Wire Wire Line
+	3700 3950 4000 3950
+Wire Wire Line
+	3000 4250 3000 4150
+Connection ~ 3000 4250
+$Comp
+L power:+3.3V #PWR0113
+U 1 1 5BA0E33D
+P 3000 3950
+F 0 "#PWR0113" H 3000 3800 50  0001 C CNN
+F 1 "+3.3V" H 3015 4123 50  0000 C CNN
+F 2 "" H 3000 3950 50  0001 C CNN
+F 3 "" H 3000 3950 50  0001 C CNN
+	1    3000 3950
+	1    0    0    -1
+$EndComp
 $EndSCHEMATC

Commit message: propozycja skonczona
Changed lines of the file:
@@
 	1    0    0    -1
 $EndComp
+Text Label 2450 1900 0    50   ~ 0
+5V_INP
 $EndSCHEMATC

Commit message: wersja produkcyjna
Parts:
- J2: footprint Connector_PinHeader_2.54mm:PinHeader_1x02_P2.54mm_Vertical -> TerminalBlock_Phoenix:TerminalBlock_Phoenix_MPT-0,5-2-2.54_1x02_P2.54mm_Horizontal
Changed lines of the file:
@@
 F 0 "J2" H 2256 2078 50  0000 C CNN
 F 1 "POWER" H 2256 1987 50  0000 C CNN
-F 2 "Connector_PinHeader_2.54mm:PinHeader_1x02_P2.54mm_Vertical" H 2150 1900 50  0001 C CNN
+F 2 "TerminalBlock_Phoenix:TerminalBlock_Phoenix_MPT-0,5-2-2.54_1x02_P2.54mm_Horizontal" H 2150 1900 50  0001 C CNN
 F 3 "~" H 2150 1900 50  0001 C CNN
 	1    2150 1900
